File: fpc_power.kicad_sch (KiCad schematic)
At the start: 22 parts, among them J2 Conn_01x02_Pin, U2 NCP1117-3.3_SOT223, U5 TLV74328_SOT23-5, U6 TLV74315_SOT23-5

Commit message: discarded 24MHz crystal. ERC passed 1st time
Parts:
- removed U2: NCP1117-3.3_SOT223, Package_TO_SOT_SMD:SOT-223-3_TabPin2, symbol Regulator_Linear:NCP1117-3.3_SOT223
- added U8: NCP1117-3.3_SOT223, Package_TO_SOT_SMD:SOT-223-3_TabPin2, symbol Regulator_Linear:NCP1117-3.3_SOT223
Connections:
- net +3V3: now also U8.2 (VO)
- net +5V: now also U8.3 (VI)
- net GND: now also U8.1 (GND)
Other:
- moved on the sheet: C36, J2

Commit message: updates in layout
Parts:
- C36: footprint Capacitor_SMD:C_0603_1608Metric_Pad1.08x0.95mm_HandSolder -> Capacitor_THT:CP_Radial_D8.0mm_P2.50mm
- J2: footprint Connector_PinHeader_2.54mm:PinHeader_1x02_P2.54mm_Vertical -> TerminalBlock:TerminalBlock_MaiXu_MX126-5.0-02P_1x02_P5.00mm
Connections:
- net +3V3 renamed +3.3V
