File: FPSP Camera.kicad_sch (KiCad schematic)
At the start: 75 parts, among them J101 Conn_01x24_Socket, J102 SM03B-SRSS-TB, J103 USB_B_Micro, J104 Conn_02x06_Odd_Even, U1 ICM-45686, U102 W25Q128JVS, U103 RP2350_60QFN, U104 TLV75533PDRV, U105 TLV73328PDRV, U106 TLV73315PDRV, Y101 SiT8008xx-1x-xxE

Commit message: Reannotated schematic
Parts:
- renumbered C123 to C1, C126 to C10, C106 to C11, C107 to C12, C127 to C13, C108 to C14, C109 to C15, C110 to C16, C128 to C17, C122 to C18, C111 to C19, C117 to C2, C112 to C20, C113 to C21, C119 to C22, C114 to C23, C115 to C24, C121 to C25, C120 to C26, C4 to C27, C5 to C28, C3 to C29, C118 to C3, C6 to C30, C101 to C4, C124 to C5, C102 to C6, C116 to C7, C103 to C8, C125 to C9, D101 to D1, D102 to D2, D103 to D3, D104 to D4, H101 to H1, H102 to H2, H103 to H3, H104 to H4, J103 to J1, J104 to J2, J102 to J3, J101 to J4, JP101 to JP1, JP102 to JP2, L101 to L1, R108 to R1, R121 to R10, R122 to R11, R123 to R12, R116 to R13, R118 to R14, R124 to R15, R3 to R16, R120 to R17, R111 to R18, R112 to R19, R104 to R2, R113 to R20, R115 to R21, R117 to R22, R119 to R3, R114 to R4, R105 to R5, R106 to R6, R109 to R7, R110 to R8, R107 to R9, TP101 to TP1, U104 to U1, U105 to U2, U103 to U3, U106 to U4, U102 to U5, U1 to U6, Y101 to Y1

Commit message: update MCU layout (initial draft)
Parts:
- removed R21: 0R, Resistor_SMD:R_0603_1608Metric_Pad0.98x0.95mm_HandSolder, symbol Device:R
- added C31, C32: 0.1u, Capacitor_SMD:C_0402_1005Metric, symbol Device:C
- added JP3: SolderJumper_2_Open, Jumper:SolderJumper-2_P1.3mm_Open_RoundedPad1.0x1.5mm, symbol Jumper:SolderJumper_2_Open
- C1, C10, C11, C12, C13, C14, C15, C16, C17, C18, C19, C2, C20, C21, C23, C24, C25, C26, C3, C4, C5, C6, C7, C8, C9: footprint Capacitor_SMD:C_0603_1608Metric_Pad1.08x0.95mm_HandSolder -> Capacitor_SMD:C_0402_1005Metric
- C27, C28, C29, C30: footprint Capacitor_SMD:C_0402_1005Metric_Pad0.74x0.62mm_HandSolder -> Capacitor_SMD:C_0402_1005Metric
- J4: footprint Connector_FFC-FPC:TE_2-84952-4_1x24-1MP_P1.0mm_Horizontal -> Connector_FFC-FPC:TE_2-1734839-3_1x23-1MP_P0.5mm_Horizontal
- R1, R10, R11, R12, R13, R14, R15, R17, R18, R19, R2, R20, R22, R3, R4, R5, R6: footprint Resistor_SMD:R_0603_1608Metric_Pad0.98x0.95mm_HandSolder -> Capacitor_SMD:C_0402_1005Metric
- R16: footprint Resistor_SMD:R_0402_1005Metric_Pad0.72x0.64mm_HandSolder -> Capacitor_SMD:C_0402_1005Metric
- U6: footprint ICM-45686:IC_ICM-45686 -> ICM_45686:IC_ICM-45686
Connections:
- net +1V5: now also C31.1
- net +2V8: now also C32.1
- net +3.3V: now also JP3.2 (B)
- net DATA1_1: now also JP3.1 (A)
- net DATA2_1: now also U3.34 (GPIO22); no longer U3.19 (GPIO15)
- net DATA6_1: now also U3.33 (GPIO21); no longer U3.18 (GPIO14)
- net DATA7_1: now also U3.32 (GPIO20); no longer U3.16 (GPIO12)
- net DATA8_1: now also U3.31 (GPIO19); no longer U3.15 (GPIO11)
- net DATA9_1: now also U3.28 (GPIO17); no longer U3.31 (GPIO19)
- net EXT_XCLK_1: now also U3.29 (GPIO18); no longer U3.32 (GPIO20)
- net GND: now also C31.2, C32.2
- net HSYNC_1: no longer U3.33 (GPIO21)
- net IMAGE_OUT_1_1: no longer U3.27 (GPIO16)
- net IMAGE_OUT_2_1: no longer U3.28 (GPIO17)
- net IMU_SCLK: now also U3.5 (GPIO3); no longer U3.4 (GPIO2)
- net IMU_SDI: now also U3.4 (GPIO2); no longer U3.5 (GPIO3)
- net IMU_SDO: now also U3.3 (GPIO1); no longer U3.7 (GPIO4)
- net INT_XCLK: no longer U3.34 (GPIO22)
- net PCLK_1: no longer U3.17 (GPIO13)
- net POSITION_OUT_1: now also U3.27 (GPIO16); no longer U3.29 (GPIO18)
- net SCL_cam_1: no longer U3.13 (GPIO9)
- net SDA_cam_1: no longer U3.12 (GPIO8)
- net VSYNC_1: no longer U3.10 (GPIO7)
- net ~{IMU_CS}: now also U3.7 (GPIO4); no longer U3.3 (GPIO1)
- net ~{RESET_1}: no longer U3.14 (GPIO10)
- new net IMAGE_OUT_1_1+: U3.16 (GPIO12)
- new net IMAGE_OUT_1_1-: U3.17 (GPIO13)
- new net IMAGE_OUT_2_1+: U3.18 (GPIO14)
- new net IMAGE_OUT_2_1-: U3.19 (GPIO15)
Other:
- note added: "HSTX: 12-19"
- moved on the sheet: C26, R17, R18, R19, R20, R22
